Commit message: Minichallenge 1     taked out static links from de URDF and declarethem in joint_state_publisher     also fixed the package.xml
    In case u see it hi Paolo (-_-)

File: ros2_ws/install/puzzlebot_sim/share/puzzlebot_sim/urdf/puzzlebot.urdf (robot description, URDF)
Before this commit: robot Puzzlebot_Jetson_Lidar_Ed., 7 links, 6 joints
Links:
- removed link map
- removed link odom
Joints:
- removed joint map_to_odom
- removed joint odom_to_base_footprint

Commit message: MiniChallenge 2     Added de STL files to the URDF of the puzzlebot

File: ros2_ws/install/puzzlebot_sim/share/puzzlebot_sim/urdf/puzzlebot.urdf (robot description, URDF)
Before this commit: robot Puzzlebot_Jetson_Lidar_Ed., 5 links, 4 joints
Links:
- added link caster_wheel_link; visual mesh filename=package://puzzlebot_sim/meshes/Puzzlebot_Caster_Wheel.stl
- link base_link: geometry visual mesh filename=package://puzzlebot_sim/meshes/Puzzlebot_Jetson_Lidar_Editi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
- link wheel_left: geometry visual mesh filename=package://puzzlebot_sim/meshes/Puzzlebot_Wheel.stl
- link wheel_right: geometry visual mesh filename=package://puzzlebot_sim/meshes/Puzzlebot_Wheel.stl
Joints:
- added joint caster_wheel_joint: type fixed, parent base_link, child caster_wheel_link, origin xyz=-0.1 0 -0.0025 rpy=0 0 0
- joint case_joint: parent base_footprint -> base_link

Commit message: Mninichallenge 3 - DONE     Just finished the 3erd Mninichallenge     added the shape drawer node which draws a square path for the puzzlebot to follow

File: ros2_ws/install/puzzlebot_sim/share/puzzlebot_sim/urdf/puzzlebot.urdf (robot description, URDF)
Before this commit: robot Puzzlebot_Jetson_Lidar_Ed., 6 links, 5 joints
Links:
- removed link case_link
Joints:
- removed joint case_joint
